File: jobs/earring-kicad-locked/input/earring.kicad_pcb (KiCad board)
At the start: 4 copper layers, 30.5 x 35.8 mm, 167 parts, among them J1 USB-C, Q1 ALS-PT19, Q10 BSS138W, Q2 CJ2101, Q3 BSS138W, Q4 LBSS84WT1G, Q5 BSS138W, Q6 BSS138W, Q7 BSS138W, Q8 CJ2101, Q9 BSS138W, SW2 PWR, U1 RP2350A, U10 TPS22913, U2 LGS4056H, U3 NCP730-3.3, U4 TPS22913, U5 USBLC6-2P6, U6 LSM6DS3TR-C, U7 W25Q16JVUXIQ, U8 74LVC2G14, U9 TPS22913, Y1 12MHz

Commit message: Jobs: blocks declared in job.json; the earring from simple-earring bb22fb7
A job now declares its blocks in job.json ("blocks": {name: {zones, parts}}), and
tools/add_block.py --job applies them to its input as KiCad groups, so they come back
whenever an input is pulled again (a block's group uuid is named, not random, so applying
it twice changes nothing). bluebuzz-kicad, earring-kicad and earring-kicad-locked declare
the RP2350's power block: the reference design's 1V1 and 3V3 pours with U1, L1 and their caps.

earring-kicad and earring-kicad-locked take the simple earring at bb22fb7, which moves 19
parts to the back to clear the area around the CPU; their leaderboard rows before today are
on 78920f1. All three jobs route at 120 s with nothing cut into the block (earring 10 open,
locked earring 11, bluebuzz 14, by KiCad after a refill), and the in-tab router routes the
grouped earring without error.

Co-Authored-By: Claude Opus 5.5 (1M context) <noreply@anthropic.com>
Parts:
- C16, C17, C18, C19, C20, C25, C29, D3, R19, R20, R21, R22, R3, R8, U2, U3, U4, U7: moved to B.Cu
- moved R10 23.2 mm to (91.2, 102.6), turned to 180 degrees
- moved C20 17.4 mm to (90.7, 103.8), turned to 0 degrees
- moved U4 16.8 mm to (91.2, 105.1)
- moved R3 14.8 mm to (102.2, 109.8), turned to 0 degrees
- moved C25 13.1 mm to (103.2, 105.7), turned to -90 degrees
- moved U7 10.8 mm to (101.5, 107.0), turned to 180 degrees
- moved D3 8.07 mm to (109.1, 104.8)
- moved R8 7.32 mm to (103.5, 107.6), turned to -90 degrees
- moved C19 5.31 mm to (96.0, 106.2), turned to -90 degrees
- moved C17 5.08 mm to (107.2, 106.9)
- moved C18 4.50 mm to (92.2, 105.8), turned to -90 degrees
- moved R22 4.01 mm to (109.0, 102.7), turned to 180 degrees
- moved R21 3.68 mm to (107.6, 103.0)
- moved U3 3.18 mm to (94.1, 106.5), turned to 180 degrees
- moved R20 2.72 mm to (109.2, 100.2)
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Routing:
- net CHRG_DONE: track 4.32 -> 0.00 mm, vias 2 -> 0
- net QSPI_SD3: vias 1 -> 0
- net QSPI_SD2: vias 1 -> 0
- net QSPI_SD1: vias 1 -> 0
- net QSPI_SD0: vias 1 -> 0
- net QSPI_SCLK: vias 1 -> 0
- net LED_EN_L: vias 1 -> 0
- net CHRG: vias 2 -> 0
- net 3V3: vias 8 -> 7

Commit message: Core: a pad without a hole that lists every copper layer has copper on its own side alone
KiCad gives an SMD or connector pad with no hole copper on its footprint's side only, whatever
its layer list says (*.Cu): nothing joins the layers through it. The router had taken *.Cu as
every layer, so a route that met such a pad on another layer was connected to the router and
open to KiCad (PCBench powerfreq, KiwiSDR). earring-kicad-locked takes the simple-earring
session's refreshed pre-route board, without the free-standing assist vias that dangled, and
routes with seed 3 (clean there).

Co-Authored-By: Claude Opus 5.5 (1M context) <noreply@anthropic.com>
Routing:
- net USB_C_DP: track 3.80 -> 1.80 mm
- net USB_DP: vias 1 -> 0
- net USB_DM: vias 1 -> 0
- net SWDIO: vias 1 -> 0
- net SWCLK: vias 1 -> 0
- net IMU_SDA: vias 2 -> 0
- net IMU_SCL: vias 1 -> 0
- net IMU_INT1: vias 1 -> 0
- net 3V3: vias 7 -> 6
